Commit message: urdf update

File: robot.urdf (robot description, URDF)
Before this commit: robot onshape, 8 links, 7 joints
Links:
- link compact_excavator_cabin_body_cmpl: mass 9732.8038980797646218 -> 9732.8038980797628028
- link part01_pin_1: mass 98.140190062279060612 -> 98.140190062279046401
- link part04: mass 132.70765933863825126 -> 132.70765933863822283
- link push_blade_bucket: mass 147.01808168083428541 -> 147.01808168083411488
Joints:
- removed joint full_arm_rotation_continuous
- removed joint lower_arm_continuous
- added joint full_arm_rotation: type revolute, parent compact_excavator_cabin_body_cmpl, child part01_pin_1, origin xyz=-0.040707723917193447405 -0.80673603465099630316 0.38039999999999996039 rpy=3.141592653589793116 4.8797124238540929311e-17 0.21446312817660284633, axis 0 0 1, limit effort=1 velocity=20
- added joint lower_arm: type revolute, parent part01_pin_1, child part02_cmpl, origin xyz=0.080000000000000265343 0.074999999999998845368 -0.15000000000000018874 rpy=-1.57079632679489678 0.62798416085350616811 -1.5707963267948996666, axis 0 0 1, limit effort=1 velocity=20
- joint plow1: origin xyz=-0.25499999999999983791 0.48800000000000004485 -0.20499999999999996003 rpy=1.570796326794896558 -1.3691259639683164284 -1.5707963267948987784 -> xyz=-0.25500000000000000444 0.48799999999999998934 -0.20500000000000001554 rpy=1.570796326794896558 -1.3195606112546156563 -1.5707963267948994446
- joint scoop1: origin xyz=0.12000000000000632383 -1.5403327562575594989 -5.7245874707234634116e-16 rpy=-3.1415926535897842342 -9.1149901341675310665e-15 -0.56975243178458789828 -> xyz=0.1200000000000036593 -1.540332756257559943 9.4368957093138305936e-16 rpy=3.1415926535897917837 7.373202369705688962e-16 -1.4390399398611677384
- joint tankBase_wheel: origin xyz=-0.25 -2.6156637754879717029e-15 -0.050000000000000086042 rpy=1.1368396176594208827e-17 2.0028574660182372206e-17 3.1212556965518580832 -> xyz=-0.25 -2.5715909255520656419e-15 -0.049999999999999961142 rpy=1.1763052875827275422e-17 1.9830083989986516138e-17 3.1020655818367162126
- joint upperToLow: origin xyz=-0.83999999999999763745 2.3549999999999999822 -0.13500000000000006439 rpy=-3.1415926535897926719 -7.4857794334601041014e-15 2.5913316311913741075 -> xyz=-0.83999999999999930278 2.3549999999999999822 -0.13500000000000023093 rpy=3.1415926535897922278 5.5237799528035288331e-15 2.4777537169378613946

Commit message: changed wheel rotation

File: robot.urdf (robot description, URDF)
Before this commit: robot onshape, 8 links, 7 joints
Links:
- added link compact_excavator_front_wheel, mass 17.64673591392957519; collision mesh filename=package:///compact_excavator_front_wheel.stl; visual mesh filename=package:///compact_excavator_front_wheel.stl
- added link compact_excavator_main_drive_wheel_cmpl, mass 35.986291345795820007; collision mesh filename=package:///compact_excavator_main_drive_wheel.stl; visual mesh filename=package:///compact_excavator_main_drive_wheel.stl
- added link compact_excavator_main_drive_wheel_cmpl_(1), mass 35.986291345795820007; collision mesh filename=package:///compact_excavator_main_drive_wheel.stl; visual mesh filename=package:///compact_excavator_main_drive_wheel.stl
- link compact_excavator_cabin_body_cmpl: mass 9732.8038980797628028 -> 9732.8038980797646218
- link compact_excavator_frame_body: mass 1357.3931058603629936 -> 476.76381190180200065; geometry collision mesh filename=package:///compact_excavator_frame_body.stl; collision mesh filename=package:///compact_excavator_front_wheel.stl
- link part02_cmpl: mass 694.1779351385806649 -> 694.17793513858077858
- link part03: mass 265.34907807560875881 -> 265.34907807560870197
- link part04: mass 132.70765933863822283 -> 132.7076593386383081
- link push_blade_bucket: mass 147.01808168083411488 -> 147.0180816808341433
Joints:
- removed joint fixedbase
- removed joint tankBase_wheel
- added joint fixed_base: type fixed, parent compact_excavator_cabin_body_cmpl, child compact_excavator_turret_cabin_roller, origin xyz=-0.25 -2.394831672112794725e-15 0.049999999999999988898 rpy=-6.5400986663891116335e-25 -1.0029564927205460558e-23 3.1415926535897926719, axis 0 0 1, limit effort=1 velocity=20
- added joint left_idle_passive_wheel: type continuous, parent compact_excavator_frame_body, child compact_excavator_front_wheel, origin xyz=-0.61299999999999998934 0.80000000000000026645 -0.2750000000000000222 rpy=1.570796326794896558 -1.0222876983448163646 -1.5707963267948941155, axis 0 0 1, limit effort=1 velocity=20
- added joint left_sprocket_wheel: type continuous, parent compact_excavator_frame_body, child compact_excavator_main_drive_wheel_cmpl_(1), origin xyz=-0.5739999999999999547 -0.80000000000000015543 -0.2750000000000000222 rpy=1.570796326794896558 -0.3547477759675310427 1.5707963267948976682, axis 0 0 1, limit effort=1 velocity=20
- added joint right_sprocket_wheel: type continuous, parent compact_excavator_frame_body, child compact_excavator_main_drive_wheel_cmpl, origin xyz=0.5739999999999999547 -0.80000000000000004441 -0.2750000000000000222 rpy=1.570796326794896558 -1.2984776443375001254 -1.5707963267948972241, axis 0 0 1, limit effort=1 velocity=20
- added joint tankSpin_wheel: type continuous, parent compact_excavator_turret_cabin_roller, child compact_excavator_frame_body, origin xyz=-0.25 -2.6052883279480892481e-15 -0.050000000000000002776 rpy=-5.5511151231419568159e-17 -1.1102230246202266528e-16 1.57079632679489678, axis 0 0 1, limit effort=1 velocity=20
- joint lower_arm: origin xyz=0.080000000000000265343 0.074999999999998845368 -0.15000000000000018874 rpy=-1.57079632679489678 0.62798416085350616811 -1.5707963267948996666 -> xyz=0.079999999999996157518 0.074999999999997291056 -0.1500000000000039635 rpy=-1.570796326794896558 0.39285813115170314935 -1.5707963267949009989
- joint plow1: origin xyz=-0.25500000000000000444 0.48799999999999998934 -0.20500000000000001554 rpy=1.570796326794896558 -1.3195606112546156563 -1.5707963267948994446 -> xyz=-0.25500000000000005995 0.4880000000000002669 -0.20500000000000001554 rpy=1.570796326794896558 -1.3195606112546109934 -1.57079632679489678
- joint scoop1: origin xyz=0.1200000000000036593 -1.540332756257559943 9.4368957093138305936e-16 rpy=3.1415926535897917837 7.373202369705688962e-16 -1.4390399398611677384 -> xyz=0.12000000000000410338 -1.5403327562575612752 9.4368957093138305936e-16 rpy=3.1415926535897917837 1.8859935444767496044e-16 -1.5963552846072552871
- joint upperToLow: origin xyz=-0.83999999999999930278 2.3549999999999999822 -0.13500000000000023093 rpy=3.1415926535897922278 5.5237799528035288331e-15 2.4777537169378613946 -> xyz=-0.84000000000000030198 2.3549999999999999822 -0.13500000000000003664 rpy=3.1415926535897922278 6.9325343981756730312e-15 2.5555644018935783635

Commit message: added final wheel joint

File: robot.urdf (robot description, URDF)
Before this commit: robot onshape, 11 links, 10 joints
Links:
- added link compact_excavator_front_wheel_2, mass 17.64673591392957519; collision mesh filename=package:///compact_excavator_front_wheel.stl; visual mesh filename=package:///compact_excavator_front_wheel.stl
- link compact_excavator_cabin_body_cmpl: mass 9732.8038980797646218 -> 9732.8038980797628028
- link compact_excavator_frame_body: mass 476.76381190180200065 -> 459.11707598787205598; geometry collision mesh filename=package:///compact_excavator_frame_body.stl; visual mesh filename=package:///compact_excavator_frame_body.stl
- link part01_pin_1: mass 98.140190062279046401 -> 98.140190062279060612
- link part02_cmpl: mass 694.17793513858077858 -> 694.17793513858055121
- link part03: mass 265.34907807560870197 -> 265.34907807560875881
- link part04: mass 132.7076593386383081 -> 132.70765933863819441
- link push_blade_bucket: mass 147.0180816808341433 -> 147.01808168083425699
Joints:
- added joint right_idle_passive_wheel: type continuous, parent compact_excavator_frame_body, child compact_excavator_front_wheel_2, origin xyz=0.54800000000000004263 0.80000000000000015543 -0.27499999999999996669 rpy=1.57079632679489678 -1.1102232252180887662e-16 -1.5707963267948976682, axis 0 0 1, limit effort=1 velocity=20

Commit message: added rollers

File: robot.urdf (robot description, URDF)
Before this commit: robot onshape, 12 links, 11 joints
Links:
- added link track_roller_wheel_1, mass 0; collision mesh filename=package:///track_roller_wheel_1.stl; visual mesh filename=package:///track_roller_wheel_1.stl
- added link track_roller_wheel_1_2, mass 0; collision mesh filename=package:///track_roller_wheel_1.stl; visual mesh filename=package:///track_roller_wheel_1.stl
- added link track_roller_wheel_1_3, mass 0; collision mesh filename=package:///track_roller_wheel_1.stl; visual mesh filename=package:///track_roller_wheel_1.stl
- added link track_roller_wheel_1_4, mass 0; collision mesh filename=package:///track_roller_wheel_1.stl; visual mesh filename=package:///track_roller_wheel_1.stl
- added link track_roller_wheel_1_5, mass 0; collision mesh filename=package:///track_roller_wheel_1.stl; visual mesh filename=package:///track_roller_wheel_1.stl
- added link track_roller_wheel_1_6, mass 0; collision mesh filename=package:///track_roller_wheel_1.stl; visual mesh filename=package:///track_roller_wheel_1.stl
- link compact_excavator_cabin_body_cmpl: mass 9732.8038980797628028 -> 9732.8038980797646218
- link compact_excavator_frame_body: mass 459.11707598787205598 -> 459.11707598787234019
- link compact_excavator_main_drive_wheel_cmpl: mass 35.986291345795820007 -> 35.986291345795812902
- link compact_excavator_main_drive_wheel_cmpl_(1): mass 35.986291345795820007 -> 35.986291345795812902
- link part02_cmpl: mass 694.17793513858055121 -> 694.17793513858077858
- link part04: mass 132.70765933863819441 -> 132.70765933863825126
- link push_blade_bucket: mass 147.01808168083425699 -> 147.01808168083420014
Joints:
- added joint roll_wheel1: type revolute, parent compact_excavator_frame_body, child track_roller_wheel_1, origin xyz=0.66300000000000003375 -0.4500000000000000111 -0.3850000000000001199 rpy=1.5707963267948972241 -0.13040282330050728676 1.5707963267948934494, axis 0 0 1, limit effort=1 velocity=20
- added joint roll_wheel2: type revolute, parent compact_excavator_frame_body, child track_roller_wheel_1_2, origin xyz=0.66300000000000003375 1.6208704515421723024e-16 -0.38499999999999995337 rpy=1.570796326794896558 0.29254554115964298555 1.5707963267948799047, axis 0 0 1, limit effort=1 velocity=20
- added joint roll_wheel3: type revolute, parent compact_excavator_frame_body, child track_roller_wheel_1_3, origin xyz=0.66299999999999992273 0.45000000000000023315 -0.38499999999999995337 rpy=1.570796326794896558 7.7715625765379412706e-16 1.5707963267948807928, axis 0 0 1, limit effort=1 velocity=20
- added joint roll_wheel4: type revolute, parent compact_excavator_frame_body, child track_roller_wheel_1_4, origin xyz=-0.66299999999999992273 -0.44999999999999995559 -0.38500000000000000888 rpy=-1.570796326794896558 7.7715625765379412706e-16 1.5707963267948807928, axis 0 0 1, limit effort=1 velocity=20
- added joint roll_wheel5: type revolute, parent compact_excavator_frame_body, child track_roller_wheel_1_5, origin xyz=-0.66300000000000003375 1.4276916718361678559e-16 -0.38500000000000000888 rpy=-1.570796326794896558 7.7715625765379412706e-16 1.5707963267948807928, axis 0 0 1, limit effort=1 velocity=20
- added joint roll_wheel6: type revolute, parent compact_excavator_frame_body, child track_roller_wheel_1_6, origin xyz=-0.66300000000000014477 0.45000000000000028866 -0.38499999999999995337 rpy=1.570796326794896558 0.67460937465725012707 -1.5707963267948736874, axis 0 0 1, limit effort=1 velocity=20

Commit message: added 2 idlers, and made rollers continuous joints.

File: robot.urdf (robot description, URDF)
Before this commit: robot onshape, 18 links, 17 joints
Links:
- added link carrier_roller, mass 4.8639330759548453642; collision mesh filename=package:///carrier_roller.stl; visual mesh filename=package:///carrier_roller.stl
- added link carrier_roller_2, mass 4.8639330759548453642; collision mesh filename=package:///carrier_roller.stl; visual mesh filename=package:///carrier_roller.stl
- link compact_excavator_frame_body: mass 459.11707598787234019 -> 459.11707598787239704
- link compact_excavator_main_drive_wheel_cmpl: mass 35.986291345795812902 -> 35.986291345795820007
- link compact_excavator_main_drive_wheel_cmpl_(1): mass 35.986291345795812902 -> 35.986291345795820007
- link compact_excavator_turret_cabin_roller: mass 72.827596459303620691 -> 72.82759645930360648
- link part04: mass 132.70765933863825126 -> 132.70765933863819441
- link push_blade_bucket: mass 147.01808168083420014 -> 147.01808168083425699
Joints:
- removed joint roll_wheel1
- removed joint roll_wheel2
- removed joint roll_wheel3
- removed joint roll_wheel4
- removed joint roll_wheel5
- removed joint roll_wheel6
- added joint idler1_wheel: type continuous, parent compact_excavator_frame_body, child carrier_roller, origin xyz=0.48399999999999998579 9.8890270385806678237e-17 -0.13000000000000047629 rpy=1.570796326794896336 0.082813481944898445497 -1.5707963267948976682, axis 0 0 1, limit effort=1 velocity=20
- added joint idler2_wheel: type continuous, parent compact_excavator_frame_body, child carrier_roller_2, origin xyz=-0.48400000000000009681 8.7258015952359919992e-17 -0.1299999999999995326 rpy=1.5707963267948950037 -1.1102232252196901538e-16 1.5707963267948976682, axis 0 0 1, limit effort=1 velocity=20
- added joint roll_wheel_1: type continuous, parent compact_excavator_frame_body, child track_roller_wheel_1, origin xyz=0.66300000000000003375 -0.4500000000000000111 -0.3850000000000001199 rpy=1.5707963267948972241 -0.13040282330050728676 1.5707963267948934494, axis 0 0 1, limit effort=1 velocity=20
- added joint roll_wheel_2: type continuous, parent compact_excavator_frame_body, child track_roller_wheel_1_2, origin xyz=0.66300000000000003375 1.6208704515421723024e-16 -0.38499999999999995337 rpy=1.570796326794896558 0.29254554115964298555 1.5707963267948799047, axis 0 0 1, limit effort=1 velocity=20
- added joint roll_wheel_3: type continuous, parent compact_excavator_frame_body, child track_roller_wheel_1_3, origin xyz=0.66299999999999992273 0.45000000000000023315 -0.38499999999999995337 rpy=1.570796326794896558 7.7715625765379412706e-16 1.5707963267948807928, axis 0 0 1, limit effort=1 velocity=20
- added joint roll_wheel_4: type continuous, parent compact_excavator_frame_body, child track_roller_wheel_1_4, origin xyz=-0.66299999999999992273 -0.44999999999999995559 -0.38500000000000000888 rpy=-1.570796326794896558 7.7715625765379412706e-16 1.5707963267948807928, axis 0 0 1, limit effort=1 velocity=20
- added joint roll_wheel_5: type continuous, parent compact_excavator_frame_body, child track_roller_wheel_1_5, origin xyz=-0.66300000000000003375 1.4276916718361678559e-16 -0.38500000000000000888 rpy=-1.570796326794896558 7.7715625765379412706e-16 1.5707963267948807928, axis 0 0 1, limit effort=1 velocity=20
- added joint roll_wheel_6: type continuous, parent compact_excavator_frame_body, child track_roller_wheel_1_6, origin xyz=-0.66300000000000014477 0.45000000000000028866 -0.38499999999999995337 rpy=1.570796326794896558 0.67460937465725012707 -1.5707963267948736874, axis 0 0 1, limit effort=1 velocity=20

Commit message: tate - added thumb part h_blade_bucket.part

File: robot.urdf (robot description, URDF)
Before this commit: robot onshape, 20 links, 19 joints
Links:
- added link excavthumb, mass 60.713348927195980309; collision mesh filename=package:///connector.stl; collision mesh filename=package:///connector.stl
- link compact_excavator_frame_body: mass 459.11707598787239704 -> 459.11707598787228335
- link compact_excavator_turret_cabin_roller: mass 72.82759645930360648 -> 72.827596459303620691
- link part03: mass 265.34907807560875881 -> 265.34907807560870197
- link part04: mass 132.70765933863819441 -> 132.60396921004004867
- link push_blade_bucket: mass 147.01808168083425699 -> 147.01808168083422856
Joints:
- added joint thumbHinge: type revolute, parent part04, child excavthumb, origin xyz=-1.207922650792170316e-13 -8.2600593032111646608e-14 -0.1150000000000003797 rpy=7.9768716782650456688e-16 1.8511064904045220139e-15 1.7510332795702965303, axis 0 0 1, limit effort=1 velocity=20
- joint full_arm_rotation: origin xyz=-0.040707723917193447405 -0.80673603465099630316 0.38039999999999996039 rpy=3.141592653589793116 4.8797124238540929311e-17 0.21446312817660284633 -> xyz=-0.040707723917193440466 -0.80673603465099630316 0.38039999999999996039 rpy=3.141592653589793116 1.3405772267554363358e-16 0.49184482936957452104
- joint lower_arm: origin xyz=0.079999999999996157518 0.074999999999997291056 -0.1500000000000039635 rpy=-1.570796326794896558 0.39285813115170314935 -1.5707963267949009989 -> xyz=0.079999999999999904521 0.074999999999999733546 -0.14999999999999980016 rpy=-1.570796326794896558 0.69362897114705091006 -1.5707963267948985564
- joint plow1: origin xyz=-0.25500000000000005995 0.4880000000000002669 -0.20500000000000001554 rpy=1.570796326794896558 -1.3195606112546109934 -1.57079632679489678 -> xyz=-0.25500000000000000444 0.48800000000000004485 -0.20500000000000001554 rpy=1.570796326794896558 -1.2607163429716079506 -1.570796326794896558
- joint scoop1: origin xyz=0.12000000000000410338 -1.5403327562575612752 9.4368957093138305936e-16 rpy=3.1415926535897917837 1.8859935444767496044e-16 -1.5963552846072552871 -> xyz=0.11999999999999966249 -1.5403327562575594989 -3.8857805861880478915e-16 rpy=3.1415926535897895633 -3.1950791765547316365e-15 -0.80531265657487949294
- joint upperToLow: origin xyz=-0.84000000000000030198 2.3549999999999999822 -0.13500000000000003664 rpy=3.1415926535897922278 6.9325343981756730312e-15 2.5555644018935783635 -> xyz=-0.83999999999999985789 2.3549999999999999822 -0.13499999999999978684 rpy=-3.1415926535897877869 -7.0950929862569758372e-15 1.2267499240314121423
